Commit message: feat: IMU激光去畸变 + EKF加速度轴修正 + IMU URDF朝向修正
新增:
- scan_deskew.py: 用 IMU ω_z 补偿扫描过程中的机器人旋转
- slam.launch: deskew 开关 + relay, gmapping 始终读 /scan_deskewed

修正:
- ekf.yaml: 加速度轴 ax→ay (IMU Y轴=车头前进方向)
- robot.urdf: imu_joint 加 rpy 旋转 (IMU Y→车头, X→右, Z→上)

文档:
- SETUP.md: 补齐 source 提示 + kill_ros 清理脚本

File: src/robot_bringup/urdf/robot.urdf (robot description, URDF)
Before this commit: robot diff_drive_robot, 7 links, 6 joints
Joints:
- joint imu_joint: origin xyz=0.05 0 0.06 -> xyz=0.05 0 0.06 rpy=0 0 -1.5708

Commit message: fix: IMU帧旋转+EKF对齐+EMA平滑+线程安全+脚本健壮性
固件 (esp32_firmware.ino):
- IMU frame_id: imu_link → base_link, 添加 R_z(π/2) 旋转
- 互补滤波 accel_roll: 修正 Z 轴符号 (atan2(-ay, az))
- 校准段 cf_roll 初始化和主循环公式保持一致

EKF (ekf.yaml):
- odom y 改为 false (差速车无法横移)
- IMU ax 改为 true (前进加速度, 对齐固件帧旋转)

跟随 (laser_follower.py):
- 添加角度 EMA 平滑, 锁定瞬间初始化避免冷启动滞后
- 移除未使用的 target_angle 变量

去畸变 (scan_deskew.py):
- 添加 threading.Lock 保护 IMU 缓冲区线程安全

雷达驱动 (s9_lidar_driver.py + tools/lidar_*):
- 移除 sudo chmod 666 硬编码, 改用 udev 规则管理权限
- 添加串口打开异常处理和用户友好的错误提示
- lidar_view: 帧解析错误不再静默吞噬, 前3次打印
- lidar_sdk_driver: 添加 SIGINT/SIGTERM 优雅退出 + serial.close()

启动脚本 (slam/nav/save_map/kill_ros):
- slam_start.sh + nav_start.sh: 添加 get_my_ip() 多网卡优先匹配
- slam_start.sh + nav_start.sh: 添加话题等待 60s 超时 + 错误提示
- nav_start.sh: 添加 /cmd_vel 冲突检测 (warn 不阻止)
- save_map.sh: 添加 set -e、source、mkdir -p
- kill_ros.sh: 新增导航/C++节点/Python节点名匹配, 更彻底清理

配置:
- URDF: base 尺寸 0.20×0.22 → 0.30×0.25
- costmap footprint: 同步更新 [-0.15,-0.125] 到 launch 和仿真
- package.xml ×2: 补全 exec_depend (gmapping/amcl/move_base/teb 等)
- CMakeLists: 移除已删除的 sim_radar.py 安装

文档:
- SETUP.md: 大规模增强 (IP 变量/腿跟踪/EKF/设备职责表/排错)
- README.md: 删除重复标题, max_vel_x 更新为 0.6
- 删除 tools/hole_reference.txt (底盘孔位参考, 已不再需要)

File: src/robot_bringup/urdf/robot.urdf (robot description, URDF)
Before this commit: robot diff_drive_robot, 7 links, 6 joints
Links:
- link base_footprint: geometry visual box size=0.30 0.25 0.02
- link base_link: geometry visual box size=0.30 0.25 0.12
